File: 8052.kicad_pcb (KiCad board)
At the start: 4 copper layers, 100 x 100 mm, 29 parts, among them J1 Conn_02x20_Odd_Even, U1 AT89C52, U10 74AHCT1G32, U2 74LS573, U3 62256, U4 DS1230AB-100+, U5 74AHCT1G00, U6 74AHCT1G32, U7 74LS138, U8 74AHCT1G00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

Commit message: making layout changes
Parts:
- added J2: Conn_01x10_Pin, Connector_PinHeader_2.54mm:PinHeader_1x10_P2.54mm_Vertical, F.Cu at (57.1, 52.4)
- J1: value Conn_02x20_Odd_Even -> Conn_02x25_Odd_Even; footprint Connector_PinHeader_2.54mm:PinHeader_2x20_P2.54mm_Vertical -> Connector_PinHeader_2.54mm:PinHeader_2x25_P2.54mm_Vertical
- moved U7 39.3 mm to (163.3, 74.6)
- moved J1 4.26 mm to (81.6, 106.3)
Connections:
- J1 pad 17: /0000H -> unconnected-(J1-Pin_17-Pad17)
- J1 pad 19: /2000H -> unconnected-(J1-Pin_19-Pad19)
- J1 pad 21: /4000H -> unconnected-(J1-Pin_21-Pad21)
- J1 pad 23: /6000H -> unconnected-(J1-Pin_23-Pad23)
- J1 pad 25: /8000H -> unconnected-(J1-Pin_25-Pad25)
- J1 pad 27: /A000H -> unconnected-(J1-Pin_27-Pad27)
- J1 pad 29: /C000H -> unconnected-(J1-Pin_29-Pad29)
- J1 pad 31: /E000H -> unconnected-(J1-Pin_31-Pad31)
Routing:
- net /ALE: track 0.00 -> 27.5 mm, vias 0 -> 1
- net /D7: track 92.5 -> 72.4 mm
- net /~{EA}: track 27.8 -> 8.35 mm
- net /D6: track 94.1 -> 75.8 mm
- net /D5: track 96.5 -> 78.9 mm
- net /D4: track 98.8 -> 82.2 mm
- net /~{PSEN}: track 31.4 -> 21.6 mm, vias 0 -> 1
- net /~{RD}: track 29.5 -> 38.6 mm, vias 0 -> 1
- net /D2: track 114.8 -> 110.8 mm, vias 5 -> 2
- net /D3: track 98.4 -> 95.5 mm
- net /A15: track 67.1 -> 69.7 mm
- net /A2: track 87.5 -> 85.7 mm
- net /A1: track 89.8 -> 88.0 mm
- net /D0: track 110.6 -> 112.3 mm
- net /A14: track 93.0 -> 94.5 mm

Commit message: update
Parts:
- J2: value Conn_01x10_Pin -> Conn_01x22_Pin; footprint Connector_PinHeader_2.54mm:PinHeader_1x10_P2.54mm_Vertical -> Connector_PinHeader_2.54mm:PinHeader_1x22_P2.54mm_Vertical
- U5, U8: moved to B.Cu
- U7: footprint Package_DIP:DIP-16_W7.62mm_Socket -> Package_SO:SOIC-16_3.9x9.9mm_P1.27mm
- moved U5 114.8 mm to (71.7, 77.5)
- moved U8 103.4 mm to (71.8, 82.8)
- moved JP2 37.1 mm to (129.4, 93.1)
- moved U7 32.6 mm to (137.4, 94.5), turned to -90 degrees
Connections:
- J1 pad 11: /ALE -> /RESET
- J1 pad 13: /~{PSEN} -> /~{WR}
- J1 pad 15: /~{EA} -> /~{RD}
- J1 pad 17: unconnected-(J1-Pin_17-Pad17) -> /ALE
- J1 pad 19: unconnected-(J1-Pin_19-Pad19) -> /~{PSEN}
- J1 pad 21: unconnected-(J1-Pin_21-Pad21) -> /~{EA}
- J1 pad 23: unconnected-(J1-Pin_23-Pad23) -> /~{RAM}
- J1 pad 25: unconnected-(J1-Pin_25-Pad25) -> /A13/RAM
- J1 pad 27: unconnected-(J1-Pin_27-Pad27) -> /~{WR_NVRAM}
- J1 pad 29: unconnected-(J1-Pin_29-Pad29) -> /~{NVRAM}
- J1 pad 31: unconnected-(J1-Pin_31-Pad31) -> /RD_ANY
- J1 pad 7: /~{WR} -> unconnected-(J1-Pin_7-Pad7)
- J1 pad 9: /~{RD} -> unconnected-(J1-Pin_9-Pad9)
Routing:
- net /~{RD}: track 38.6 -> 81.7 mm, vias 1 -> 3
- net /~{PSEN}: track 21.6 -> 47.0 mm
- net /ALE: track 27.5 -> 47.1 mm
- net /~{EA}: track 8.35 -> 26.3 mm, vias 0 -> 1
- net /D7: track 72.4 -> 87.1 mm
- net /~{WR}: track 29.2 -> 42.6 mm, vias 0 -> 1
- net /D6: track 75.8 -> 88.6 mm
- net /D5: track 78.9 -> 89.8 mm
- net /D4: track 82.2 -> 91.3 mm
- net /D0: track 112.3 -> 117.1 mm
- net /A11: track 105.1 -> 109.5 mm
- net /D1: track 111.2 -> 115.3 mm
- net /A9: track 100.7 -> 104.5 mm
- net /A12: track 99.7 -> 103.4 mm
- net /A7: track 84.9 -> 81.2 mm
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
Commit message: update
Parts:
- C3, C4: moved to B.Cu
- moved JP2 37.3 mm to (93.6, 82.7)
- moved C4 5.94 mm to (73.8, 107.8), turned to 180 degrees
- moved C3 5.50 mm to (63.7, 107.8)
- moved U7 4.37 mm to (136.8, 98.8)
- moved J1 3.81 mm to (81.5, 110.1)
Connections:
- J1 pad 11: /RESET -> /~{RD}
- J1 pad 13: /~{WR} -> /ALE
- J1 pad 15: /~{RD} -> /~{PSEN}
- J1 pad 17: /ALE -> /~{EA}
- J1 pad 19: /~{PSEN} -> /~{RAM}
- J1 pad 21: /~{EA} -> /A13/RAM
- J1 pad 23: /~{RAM} -> /~{WR_NVRAM}
- J1 pad 25: /A13/RAM -> /~{NVRAM}
- J1 pad 27: /~{WR_NVRAM} -> /RD_ANY
- J1 pad 29: /~{NVRAM} -> unconnected-(J1-Pin_29-Pad29)
- J1 pad 31: /RD_ANY -> unconnected-(J1-Pin_31-Pad31)
- J1 pad 41: unconnected-(J1-Pin_41-Pad41) -> /E000H
- J1 pad 42: unconnected-(J1-Pin_42-Pad42) -> /C000H
- J1 pad 5: unconnected-(J1-Pin_5-Pad5) -> /CLK_EXT
- J1 pad 7: unconnected-(J1-Pin_7-Pad7) -> /RESET
- J1 pad 9: unconnected-(J1-Pin_9-Pad9) -> /~{WR}
Routing:
- net /0000H: track 0.00 -> 81.5 mm, vias 0 -> 2
- net /RESET: track 0.00 -> 56.6 mm, vias 0 -> 1
- net /~{RAM}: track 24.2 -> 67.9 mm, vias 1 -> 4
- net /~{EA}: track 26.3 -> 51.4 mm
- net /A15: track 71.7 -> 95.0 mm
- net /A13: track 90.3 -> 113.1 mm
- net /A14: track 95.3 -> 117.9 mm, vias 1 -> 2
- net /E000H: track 0.00 -> 18.7 mm, vias 0 -> 1
- net /D7: track 87.1 -> 96.2 mm, vias 1 -> 3
- net /D6: track 88.6 -> 96.6 mm, vias 1 -> 3
- net /~{RD}: track 81.7 -> 89.3 mm
- net /A11: track 109.5 -> 117.0 mm
- net /D5: track 89.8 -> 96.6 mm, vias 1 -> 3
- net /C000H: track 0.00 -> 6.32 mm, vias 0 -> 1
- net /D4: track 91.3 -> 97.0 mm, vias 1 -> 3
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Other:
- board size 100 x 100 mm -> 93 x 63 mm

Commit message: update
Parts:
- removed C7, C8, C9: C0805_100nF_16V_X7R, Capacitor_SMD:C_0805_2012Metric
- removed U5, U8, U9: 74AHCT1G00, Package_TO_SOT_SMD:SOT-23-5
- added H1: MountingHole, MountingHole:MountingHole_3.2mm_M3, F.Cu at (144.5, 49.5)
- added H2: MountingHole, MountingHole:MountingHole_3.2mm_M3, F.Cu at (56.5, 108.5)
- added H3: MountingHole, MountingHole:MountingHole_3.2mm_M3, F.Cu at (56.5, 49.5)
- added H4: MountingHole, MountingHole:MountingHole_3.2mm_M3, F.Cu at (144.5, 108.5)
- added J3: Conn_01x20_Pin, Connector_PinHeader_2.54mm:PinHeader_1x20_P2.54mm_Vertical, F.Cu at (145.0, 54.9)
- added R1: R0805_10k_1%_125mW_100PPM_AC, Resistor_SMD:R_0805_2012Metric, F.Cu at (125.0, 101.3)
- added U11: 74HCT00, Package_SO:SO-14_3.9x8.65mm_P1.27mm, B.Cu at (68.5, 85.3)
- C10, C11, C12: moved to B.Cu
- J2: value Conn_01x22_Pin -> Conn_01x20_Pin; footprint Connector_PinHeader_2.54mm:PinHeader_1x22_P2.54mm_Vertical -> Connector_PinHeader_2.54mm:PinHeader_1x20_P2.54mm_Vertical
- moved JP1 91.2 mm to (87.0, 82.9)
- moved JP3 81.9 mm to (83.2, 82.9)
- moved C11 72.2 mm to (138.1, 102.2), turned to 90 degrees
- moved C12 69.4 mm to (126.1, 93.8)
- moved U10 68.0 mm to (129.3, 92.5), turned to 180 degrees
- moved C10 64.6 mm to (134.0, 92.3), turned to -90 degrees
- moved U6 61.5 mm to (135.2, 92.5), turned to 180 degrees
- moved U7 3.56 mm to (133.2, 98.8)
- moved J1 3.52 mm to (78.0, 110.0)
- moved J2 2.74 mm to (56.0, 55.0)
- moved C3 2.12 mm to (61.6, 107.8)
- moved C4 2.12 mm to (71.7, 107.8)
- moved Y1 2.12 mm to (69.1, 107.8)
- moved C6 1.91 mm to (123.1, 90.9), turned to 180 degrees
- moved JP2 0.15 mm to (93.6, 82.9)
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Connections:
- J1 pad 29: unconnected-(J1-Pin_29-Pad29) -> /CS_EX_ROM
- J1 pad 31: unconnected-(J1-Pin_31-Pad31) -> /DECODER
- J1 pad 43: unconnected-(J1-Pin_43-Pad43) -> /A000H
- J1 pad 44: unconnected-(J1-Pin_44-Pad44) -> /8000H
- J1 pad 45: unconnected-(J1-Pin_45-Pad45) -> /6000H
- J1 pad 46: unconnected-(J1-Pin_46-Pad46) -> /4000H
- J1 pad 47: unconnected-(J1-Pin_47-Pad47) -> /2000H
- J1 pad 48: unconnected-(J1-Pin_48-Pad48) -> /0000H
- J1 pad 49: unconnected-(J1-Pin_49-Pad49) -> GND
- J1 pad 50: unconnected-(J1-Pin_50-Pad50) -> +5V
- J2 pad 1: unconnected-(J2-Pin_1-Pad1) -> /P1.0
- J2 pad 10: unconnected-(J2-Pin_10-Pad10) -> /P3.0/RXD
- J2 pad 11: /P3.0/RXD -> /P3.1/TXD
- J2 pad 12: /P3.1/TXD -> /P3.2/~{INT0}
- J2 pad 13: /P3.2/~{INT0} -> /P3.3/~{INT1}
- J2 pad 14: /P3.3/~{INT1} -> /P3.4/T0
- J2 pad 15: /P3.4/T0 -> /P3.5/T1
- J2 pad 16: /P3.5/T1 -> /~{WR}
- J2 pad 17: /~{WR} -> /~{RD}
- J2 pad 18: /~{RD} -> GND
- J2 pad 19: unconnected-(J2-Pin_19-Pad19) -> +5V
- J2 pad 2: /P1.0 -> /P1.1
- J2 pad 20: unconnected-(J2-Pin_20-Pad20) -> +5V
- J2 pad 3: /P1.1 -> /P1.2/PWM
- J2 pad 4: /P1.2/PWM -> /P1.3/~{ALEDIS}
- J2 pad 5: /P1.3/~{ALEDIS} -> /P1.4/~{PMGPULSE}
- J2 pad 6: /P1.4/~{PMGPULSE} -> /P1.5/~{PGMEN}
- J2 pad 7: /P1.5/~{PGMEN} -> /P1.6/~{DMA_ACK}
- J2 pad 8: /P1.6/~{DMA_ACK} -> /P1.7/~{LTP}
- J2 pad 9: /P1.7/~{LTP} -> GND
- U7 pad 6: +5V -> /DECODER
Routing:
- net /RD_ANY: track 0.00 -> 107.0 mm, vias 0 -> 3
- net /~{NVRAM}: track 0.00 -> 82.4 mm, vias 0 -> 2
- net /RESET: track 56.6 -> 118.4 mm, vias 1 -> 4
- net /~{WR_NVRAM}: track 0.00 -> 60.7 mm, vias 0 -> 1
- net Net-(JP1-B): track 0.00 -> 44.6 mm, vias 0 -> 1
- net /CS_EX_ROM: track 0.00 -> 41.2 mm, vias 0 -> 1
- net /~{LD}: track 0.00 -> 40.1 mm, vias 0 -> 1
- net /~{WR}: track 46.6 -> 85.7 mm, vias 1 -> 4
- net /A13/RAM: track 4.41 -> 37.6 mm, vias 0 -> 1
- net /DECODER: track 0.00 -> 33.2 mm, vias 0 -> 3
- net /P1.3/~{ALEDIS}: track 4.01 -> 34.0 mm
- net /P1.4/~{PMGPULSE}: track 4.01 -> 34.0 mm
- net /8000H: track 0.00 -> 17.5 mm, vias 0 -> 2
- net GND: track 0.00 -> 15.0 mm, vias 0 -> 13
- net Net-(U1-XTAL2): track 0.00 -> 14.7 mm
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- added copper zone on In2.Cu, net +5V
Other:
- board size 93 x 63 mm -> 95 x 66 mm
