File: 8052.kicad_sch (KiCad schematic)
At the start: 29 parts, among them J1 Conn_02x20_Odd_Even, U1 AT89C52, U10 74AHCT1G32, U2 74LS573, U3 62256, U4 DS1230AB-100+, U5 74AHCT1G00, U6 74AHCT1G32, U7 74LS138, U8 74AHCT1G00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

Commit message: making layout changes
Parts:
- added J2: Conn_01x10_Pin, Connector_PinHeader_2.54mm:PinHeader_1x10_P2.54mm_Vertical, symbol Connector:Conn_01x10_Pin
- J1: value Conn_02x20_Odd_Even -> Conn_02x25_Odd_Even; footprint Connector_PinHeader_2.54mm:PinHeader_2x20_P2.54mm_Vertical -> Connector_PinHeader_2.54mm:PinHeader_2x25_P2.54mm_Vertical; symbol Connector_Generic:Conn_02x20_Odd_Even -> Connector_Generic:Conn_02x25_Odd_Even
Connections:
- net 0000H: no longer J1.17 (Pin_17)
- net 2000H: no longer J1.19 (Pin_19)
- net 4000H: no longer J1.21 (Pin_21)
- net 6000H: no longer J1.23 (Pin_23)
- net 8000H: no longer J1.25 (Pin_25)
- net A000H: no longer J1.27 (Pin_27)
- net C000H: no longer J1.29 (Pin_29)
- net E000H: no longer J1.31 (Pin_31)
- net P1.0: now also J2.2 (Pin_2)
- net P1.1: now also J2.3 (Pin_3)
- net P1.2/PWM: now also J2.4 (Pin_4)
- net P1.3/~{ALEDIS}: now also J2.5 (Pin_5)
- net P1.4/~{PMGPULSE}: now also J2.6 (Pin_6)
- net P1.5/~{PGMEN}: now also J2.7 (Pin_7)
- net P1.6/~{DMA_ACK}: now also J2.8 (Pin_8)
- net P1.7/~{LTP}: now also J2.9 (Pin_9)
Other:
- moved on the sheet: C10, C11, C12, C7, C8, C9, U7

Commit message: update
Parts:
- J2: value Conn_01x10_Pin -> Conn_01x22_Pin; footprint Connector_PinHeader_2.54mm:PinHeader_1x10_P2.54mm_Vertical -> Connector_PinHeader_2.54mm:PinHeader_1x22_P2.54mm_Vertical; symbol Connector:Conn_01x10_Pin -> Connector:Conn_01x22_Pin
- U7: footprint Package_DIP:DIP-16_W7.62mm_Socket -> Package_SO:SOIC-16_3.9x9.9mm_P1.27mm
Connections:
- net A13/RAM: now also J1.25 (Pin_25)
- net ALE: now also J1.17 (Pin_17); no longer J1.11 (Pin_11)
- net P3.0/RXD: now also J2.11 (Pin_11)
- net P3.1/TXD: now also J2.12 (Pin_12)
- net P3.2/~{INT0}: now also J2.13 (Pin_13)
- net P3.3/~{INT1}: now also J2.14 (Pin_14)
- net P3.4/T0: now also J2.15 (Pin_15)
- net P3.5/T1: now also J2.16 (Pin_16)
- net RD_ANY: now also J1.31 (Pin_31)
- net RESET: now also J1.11 (Pin_11)
- net ~{EA}: now also J1.21 (Pin_21); no longer J1.15 (Pin_15)
- net ~{NVRAM}: now also J1.29 (Pin_29)
- net ~{PSEN}: now also J1.19 (Pin_19); no longer J1.13 (Pin_13)
- net ~{RAM}: now also J1.23 (Pin_23)
- net ~{RD}: now also J1.15 (Pin_15), J2.18 (Pin_18); no longer J1.9 (Pin_9)
- net ~{WR_NVRAM}: now also J1.27 (Pin_27)
- net ~{WR}: now also J1.13 (Pin_13), J2.17 (Pin_17); no longer J1.7 (Pin_7)

Commit message: update
Connections:
- net A13/RAM: now also J1.21 (Pin_21); no longer J1.25 (Pin_25)
- net ALE: now also J1.13 (Pin_13); no longer J1.17 (Pin_17)
- net C000H: now also J1.42 (Pin_42)
- net E000H: now also J1.41 (Pin_41)
- net RD_ANY: now also J1.27 (Pin_27); no longer J1.31 (Pin_31)
- net RESET: now also J1.7 (Pin_7); no longer J1.11 (Pin_11)
- net ~{EA}: now also J1.17 (Pin_17); no longer J1.21 (Pin_21)
- net ~{NVRAM}: now also J1.25 (Pin_25); no longer J1.29 (Pin_29)
- net ~{PSEN}: now also J1.15 (Pin_15); no longer J1.19 (Pin_19)
- net ~{RAM}: now also J1.19 (Pin_19); no longer J1.23 (Pin_23)
- net ~{RD}: now also J1.11 (Pin_11); no longer J1.15 (Pin_15)
- net ~{WR_NVRAM}: now also J1.23 (Pin_23); no longer J1.27 (Pin_27)
- net ~{WR}: now also J1.9 (Pin_9); no longer J1.13 (Pin_13)
- net CLK_EXT: now reaches J1.5 (Pin_5)

Commit message: update
Parts:
- removed C7, C8, C9: C0805_100nF_16V_X7R, Capacitor_SMD:C_0805_2012Metric, symbol Capacitors_SMD_0805:C0805_100nF_16V_X7R
- removed U5, U8, U9: 74AHCT1G00, Package_TO_SOT_SMD:SOT-23-5, symbol 74xGxx:74AHCT1G00
- added H1, H2, H3, H4: MountingHole, MountingHole:MountingHole_3.2mm_M3, symbol Mechanical:MountingHole
- added J3: Conn_01x20_Pin, Connector_PinHeader_2.54mm:PinHeader_1x20_P2.54mm_Vertical, symbol Connector:Conn_01x20_Pin
- added R1: R0805_10k_1%_125mW_100PPM_AC, Resistor_SMD:R_0805_2012Metric, symbol Resistors_SMD_0805:R0805_10k_1%_125mW_100PPM_AC
- added U11: 74HCT00, Package_SO:SO-14_3.9x8.65mm_P1.27mm, symbol 74xx:74HCT00
- J2: value Conn_01x22_Pin -> Conn_01x20_Pin; footprint Connector_PinHeader_2.54mm:PinHeader_1x22_P2.54mm_Vertical -> Connector_PinHeader_2.54mm:PinHeader_1x20_P2.54mm_Vertical; symbol Connector:Conn_01x22_Pin -> Connector:Conn_01x20_Pin
Connections:
- net +5V: now also J1.50 (Pin_50), J2.19 (Pin_19), J2.20 (Pin_20), R1.1; no longer U7.6 (E3)
- net 0000H: now also J1.48 (Pin_48)
- net 2000H: now also J1.47 (Pin_47)
- net 4000H: now also J1.46 (Pin_46)
- net 6000H: now also J1.45 (Pin_45)
- net 8000H: now also J1.44 (Pin_44)
- net A000H: now also J1.43 (Pin_43)
- net ALE: now also U11.1
- net CS_EX_ROM: now also J1.29 (Pin_29)
- net GND: now also J1.49 (Pin_49), J2.18 (Pin_18), J2.9 (Pin_9)
- net P1.0: now also J2.1 (Pin_1); no longer J2.2 (Pin_2)
- net P1.1: now also J2.2 (Pin_2); no longer J2.3 (Pin_3)
- net P1.2/PWM: now also J2.3 (Pin_3); no longer J2.4 (Pin_4)
- net P1.3/~{ALEDIS}: now also J2.4 (Pin_4), U11.2; no longer J2.5 (Pin_5)
- net P1.4/~{PMGPULSE}: now also J2.5 (Pin_5), U11.10; no longer J2.6 (Pin_6)
- net P1.5/~{PGMEN}: now also J2.6 (Pin_6); no longer J2.7 (Pin_7)
- net P1.6/~{DMA_ACK}: now also J2.7 (Pin_7); no longer J2.8 (Pin_8)
- net P1.7/~{LTP}: now also J2.8 (Pin_8); no longer J2.9 (Pin_9)
- net P3.0/RXD: now also J2.10 (Pin_10); no longer J2.11 (Pin_11)
- net P3.1/TXD: now also J2.11 (Pin_11); no longer J2.12 (Pin_12)
- net P3.2/~{INT0}: now also J2.12 (Pin_12); no longer J2.13 (Pin_13)
- net P3.3/~{INT1}: now also J2.13 (Pin_13); no longer J2.14 (Pin_14)
- net P3.4/T0: now also J2.14 (Pin_14); no longer J2.15 (Pin_15)
- net P3.5/T1: now also J2.15 (Pin_15); no longer J2.16 (Pin_16)
- net RD_ANY: now also U11.6
- net ~{LD}: now also U11.3
- net ~{PSEN}: now also U11.4
- net ~{RD}: now also J2.17 (Pin_17), U11.5; no longer J2.18 (Pin_18)
- net ~{WR}: now also J2.16 (Pin_16), U11.9; no longer J2.17 (Pin_17)
- net DECODER: now reaches J1.31 (Pin_31)
- net DECODER: now also U7.6 (E3), R1.2
- net at JP1.3 (B): now also U11.8
Other:
- moved on the sheet: C11
