File: 8052-MCU.kicad_pcb (KiCad board)
At the start: 4 copper layers, 95 x 66 mm, 31 parts, among them J1 Conn_02x25_Odd_Even, J2 Conn_01x20_Pin, J3 Conn_01x20_Pin, U1 AT89C52, U10 74AHCT1G32, U11 74HCT00, U2 74LS573, U3 62256, U4 DS1230AB-100+, U6 74AHCT1G32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

Commit message: Renamed
Parts:
- moved H1 4.00 mm to (144.5, 45.5)
- moved H3 4.00 mm to (56.5, 45.5)
Other:
- board size 95 x 66 mm -> 95 x 70 mm
Changed lines of the file:
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@@
   )
   (footprint "MountingHole:MountingHole_3.2mm_M3" (layer "F.Cu")
-    (at 144.5 49.5)
+    (at 144.5 45.5)
     (descr "Mounting Hole 3.2mm, no annular, M3")
     (tags "mounting hole 3.2mm no annular m3")
@@
   )
   (footprint "MountingHole:MountingHole_3.2mm_M3" (layer "F.Cu")
-    (at 56.5 49.5)
+    (at 56.5 45.5)
     (descr "Mounting Hole 3.2mm, no annular, M3")
     (tags "mounting hole 3.2mm no annular m3")
@@
     )
   )
-  (gr_line (start 148 46) (end 148 112)
+  (gr_line (start 148 42) (end 148 112)
     (stroke (width 0.1) (type solid)) (layer "Edge.Cuts"))
-  (gr_line (start 53 112) (end 53 46)
+  (gr_line (start 53 112) (end 53 42)
     (stroke (width 0.1) (type solid)) (layer "Edge.Cuts"))
   (gr_line (start 148 112) (end 53 112)
     (stroke (width 0.1) (type solid)) (layer "Edge.Cuts"))
-  (gr_line (start 53 46) (end 148 46)
+  (gr_line (start 53 42) (end 148 42)
     (stroke (width 0.1) (type solid)) (layer "Edge.Cuts"))
   (segment (start 64.195 103.815) (end 64.195 107.8) (width 0.2) (layer "F.Cu") (net 1))

Commit message: update
Other:
- rule pad_to_mask_clearance: 0 -> 0.075
Changed lines of the file:
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@@
 (kicad_pcb (version 20221018) (generator pcbnew)
   (general
-    (thickness 4.69)
+    (thickness 0.917)
   )
   (paper "A4")
   (layers
     (0 "F.Cu" signal)
-    (1 "In1.Cu" signal)
+    (1 "In1.Cu" power)
     (2 "In2.Cu" signal)
     (31 "B.Cu" signal)
@@
     (48 "B.Fab" user)
     (49 "F.Fab" user)
-    (50 "User.1" user)
-    (51 "User.2" user)
-    (52 "User.3" user)
-    (53 "User.4" user)
-    (54 "User.5" user)
-    (55 "User.6" user)
-    (56 "User.7" user)
-    (57 "User.8" user)
-    (58 "User.9" user)
   )
   (setup
@@
       (layer "F.Mask" (type "Top Solder Mask") (thickness 0.01))
       (layer "F.Cu" (type "copper") (thickness 0.035))
-      (layer "dielectric 1" (type "core") (thickness 1.51) (material "FR4") (epsilon_r 4.5) (loss_tangent 0.02))
-      (layer "In1.Cu" (type "copper") (thickness 0.035))
-      (layer "dielectric 2" (type "prepreg") (thickness 1.51) (material "FR4") (epsilon_r 4.5) (loss_tangent 0.02))
-      (layer "In2.Cu" (type "copper") (thickness 0.035))
-      (layer "dielectric 3" (type "core") (thickness 1.51) (material "FR4") (epsilon_r 4.5) (loss_tangent 0.02))
+      (layer "dielectric 1" (type "prepreg") (thickness 0.1 locked) (material "FR4") (epsilon_r 4.05) (loss_tangent 0.02))
+      (layer "In1.Cu" (type "copper") (thickness 0.0175))
+      (layer "dielectric 2" (type "core") (thickness 0.565 locked) (material "FR4") (epsilon_r 4.6) (loss_tangent 0.02))
+      (layer "In2.Cu" (type "copper") (thickness 0.0175))
+      (layer "dielectric 3" (type "prepreg") (thickness 0.127 locked) (material "FR4") (epsilon_r 4.25) (loss_tangent 0.02))
       (layer "B.Cu" (type "copper") (thickness 0.035))
       (layer "B.Mask" (type "Bottom Solder Mask") (thickness 0.01))
       (layer "B.Paste" (type "Bottom Solder Paste"))
       (layer "B.SilkS" (type "Bottom Silk Screen"))
-      (copper_finish "None")
+      (copper_finish "HAL lead-free")
       (dielectric_constraints no)
+      (edge_connector yes)
     )
-    (pad_to_mask_clearance 0)
+    (pad_to_mask_clearance 0.075)
     (pcbplotparams
       (layerselection 0x00010fc_ffffffff)
@@
     (polygon
       (pts
-        (xy 53 46)
+        (xy 53 42)
         (xy 53 112)
         (xy 148 112)
-        (xy 148 46)
+        (xy 148 42)
       )
     )
@@
     (polygon
       (pts
-        (xy 53 46)
+        (xy 53 42)
         (xy 53 112)
         (xy 148 112)
-        (xy 148 46)
+        (xy 148 42)
       )
     )

Commit message: update
Parts:
- added U5: 23LC512, Package_SO:SOIC-8_3.9x4.9mm_P1.27mm, F.Cu at (41.6, 65.7)
- added U8: 23LC512, Package_SO:SOIC-8_3.9x4.9mm_P1.27mm, F.Cu at (41.6, 72.2)

Commit message: update
Parts:
- U5, U8: moved to B.Cu
- moved U5 27.9 mm to (68.7, 58.9), turned to 180 degrees
- moved U8 27.6 mm to (68.5, 65.7), turned to 180 degrees
Connections:
- net /P1.4/~{PMGPULSE} renamed /P1.4/~{PMGPULSE}/~{SS}
- J2 pad 6: /P1.5/~{PGMEN} -> /P1.5/~{PGMEN}/MOSI
- J2 pad 7: /P1.6/~{DMA_ACK} -> /P1.6/~{DMA_ACK}/MISO
- J2 pad 8: /P1.7/~{LTP} -> /P1.7/~{LTP}/SCK
- U1 pad 6: /P1.5/~{PGMEN} -> /P1.5/~{PGMEN}/MOSI
- U1 pad 7: /P1.6/~{DMA_ACK} -> /P1.6/~{DMA_ACK}/MISO
- U1 pad 8: /P1.7/~{LTP} -> /P1.7/~{LTP}/SCK
- U5 pad 2: Net-(U5-DO(IO1)) -> /P1.6/~{DMA_ACK}/MISO
- U5 pad 5: Net-(U5-DI(IO0)) -> /P1.5/~{PGMEN}/MOSI
- U5 pad 6: Net-(U5-CLK) -> /P1.7/~{LTP}/SCK
- U8 pad 2: Net-(U5-DO(IO1)) -> /P1.6/~{DMA_ACK}/MISO
- U8 pad 5: Net-(U5-DI(IO0)) -> /P1.5/~{PGMEN}/MOSI
- U8 pad 6: Net-(U5-CLK) -> /P1.7/~{LTP}/SCK
Routing:
- net unconnected-(U8-IO3-Pad7): track 0.00 -> 34.0 mm
- net /P1.4/~{PMGPULSE}/~{SS}: track 34.0 -> 0.00 mm
- net /P1.7/~{LTP}/SCK: track 0.00 -> 5.12 mm
- net /P1.7/~{LTP}: track 5.12 -> 0.00 mm
- net /P1.6/~{DMA_ACK}/MISO: track 0.00 -> 5.12 mm
- net /P1.6/~{DMA_ACK}: track 5.12 -> 0.00 mm
- net /P1.5/~{PGMEN}/MOSI: track 0.00 -> 5.12 mm
- net /P1.5/~{PGMEN}: track 5.12 -> 0.00 mm
Other:
- board text added: "8052-MCU V${REVISION}"
- board text added: "JKBI"

Commit message: update
Parts:
- added J4: Conn_02x40_Top_Bottom, Connector_PinHeader_2.54mm:PinHeader_2x40_P2.54mm_Vertical, F.Cu at (55.0, 116.5)
Other:
- board size 95 x 70 mm -> 103 x 78.3 mm
