File: 8052-MCU.kicad_sch (KiCad schematic)
At the start: 31 parts, among them J1 Conn_02x25_Odd_Even, J2 Conn_01x20_Pin, J3 Conn_01x20_Pin, U1 AT89C52, U10 74AHCT1G32, U11 74HCT00, U2 74LS573, U3 62256, U4 DS1230AB-100+, U6 74AHCT1G32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

Commit message: update
Parts:
- added U5, U8: 23LC512, Package_SO:SOIC-8_3.9x4.9mm_P1.27mm, symbol 8051_mcu_lib:23LC512
Connections:
- net +5V: now also U5.8 (VCC), U8.8 (VCC)
- net GND: now also U5.4 (GND), U8.4 (GND)
- new net: U5.2 (DO(IO1)), U8.2 (DO(IO1))
- new net: U5.5 (DI(IO0)), U8.5 (DI(IO0))
- new net: U5.6 (CLK), U8.6 (CLK)
- no-connect marks 0 -> 24
Other:
- title: (none) -> 8052-MCU

Commit message: update
Connections:
- net P1.5/~{PGMEN} is gone; now on net P1.5/~{PGMEN}/MOSI: J2.6 (Pin_6), U1.6 (P1.5)
- net P1.6/~{DMA_ACK} is gone; now on net P1.6/~{DMA_ACK}/MISO: J2.7 (Pin_7), U1.7 (P1.6)
- net P1.7/~{LTP} is gone; now on net P1.7/~{LTP}/SCK: J2.8 (Pin_8), U1.8 (P1.7)
- net P1.6/~{DMA_ACK}/MISO: now reaches U5.2 (DO(IO1)), U8.2 (DO(IO1))
- net P1.5/~{PGMEN}/MOSI: now reaches U5.5 (DI(IO0)), U8.5 (DI(IO0))
- net P1.7/~{LTP}/SCK: now reaches U5.6 (CLK), U8.6 (CLK)
- net P1.4/~{PMGPULSE} renamed P1.4/~{PMGPULSE}/~{SS}
Changed lines of the file:
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@@
   (junction (at 184.785 31.75) (diameter 0) (color 0 0 0 0)
   )
+  (junction (at 69.85 205.74) (diameter 0) (color 0 0 0 0)
+  )
   (junction (at 344.805 57.15) (diameter 0) (color 0 0 0 0)
   )
@@
   (junction (at 208.28 46.355) (diameter 0) (color 0 0 0 0)
   )
+  (junction (at 73.025 208.28) (diameter 0) (color 0 0 0 0)
+  )
   (junction (at 271.145 46.355) (diameter 0) (color 0 0 0 0)
   )
@@
   (junction (at 354.965 67.31) (diameter 0) (color 0 0 0 0)
   )
+  (junction (at 76.2 210.82) (diameter 0) (color 0 0 0 0)
+  )
   (no_connect (at 43.815 158.75))
   (no_connect (at 43.815 140.97))
@@
     (stroke (width 0) (type default))
   )
-  (wire (pts (xy 127.635 170.815) (xy 143.51 170.815))
+  (wire (pts (xy 124.46 170.815) (xy 143.51 170.815))
     (stroke (width 0) (type default))
   )
@@
     (stroke (width 0) (type default))
   )
+  (wire (pts (xy 69.85 205.74) (xy 46.355 205.74))
+    (stroke (width 0) (type default))
+  )
   (wire (pts (xy 119.38 88.9) (xy 135.255 88.9))
     (stroke (width 0) (type default))
@@
     (stroke (width 0) (type default))
   )
-  (wire (pts (xy 127.635 165.735) (xy 143.51 165.735))
-    (stroke (width 0) (type default))
-  )
   (bus (pts (xy 377.825 64.77) (xy 377.825 62.23))
     (stroke (width 0) (type default))
@@
     (stroke (width 0) (type default))
   )
+  (wire (pts (xy 73.025 208.28) (xy 46.355 208.28))
+    (stroke (width 0) (type default))
+  )
   (bus (pts (xy 231.775 60.96) (xy 231.775 63.5))
     (stroke (width 0) (type default))
@@
     (stroke (width 0) (type default))
   )
+  (wire (pts (xy 76.2 210.82) (xy 46.355 210.82))
+    (stroke (width 0) (type default))
+  )
   (wire (pts (xy 336.55 110.49) (xy 346.075 110.49))
     (stroke (width 0) (type default))
@@
     (stroke (width 0) (type default))
   )
+  (wire (pts (xy 124.46 165.735) (xy 143.51 165.735))
+    (stroke (width 0) (type default))
+  )
   (wire (pts (xy 88.9 60.96) (xy 81.28 60.96))
     (stroke (width 0) (type default))
@@
     (effects (font (size 1.27 1.27)) (justify right bottom))
   )
-  (label "P1.4{slash}~{PMGPULSE}" (at 43.815 78.74 180) (fields_autoplaced)
+  (label "P1.4{slash}~{PMGPULSE}{slash}~{SS}" (at 43.815 78.74 180) (fields_autoplaced)
     (effects (font (size 1.27 1.27)) (justify right bottom))
   )
@@
     (effects (font (size 1.27 1.27)) (justify right bottom))
   )
+  (label "P1.4{slash}~{PMGPULSE}{slash}~{SS}" (at 42.672 202.946 180) (fields_autoplaced)
+    (effects (font (size 1.27 1.27)) (justify right bottom))
+  )
   (label "P1.3{slash}~{ALEDIS}" (at 43.815 76.2 180) (fields_autoplaced)
     (effects (font (size 1.27 1.27)) (justify right bottom))
@@
     (effects (font (size 1.27 1.27)) (justify right bottom))
   )
-  (label "P1.7{slash}~{LTP}" (at 69.85 83.82 0) (fields_autoplaced)
-    (effects (font (size 1.27 1.27)) (justify left bottom))
-  )
   (label "P1.3{slash}~{ALEDIS}" (at 69.85 73.66 0) (fields_autoplaced)
     (effects (font (size 1.27 1.27)) (justify left bottom))
@@
     (effects (font (size 1.27 1.27)) (justify right bottom))
   )
-  (label "P1.5{slash}~{PGMEN}" (at 69.85 78.74 0) (fields_autoplaced)
-    (effects (font (size 1.27 1.27)) (justify left bottom))
-  )
-  (label "P1.7{slash}~{LTP}" (at 43.815 86.36 180) (fields_autoplaced)
+  (label "P1.7{slash}~{LTP}{slash}SCK" (at 43.815 86.36 180) (fields_autoplaced)
     (effects (font (size 1.27 1.27)) (justify right bottom))
   )
@@
     (effects (font (size 1.27 1.27)) (justify left bottom))
   )
-  (label "P1.4{slash}~{PMGPULSE}" (at 69.85 76.2 0) (fields_autoplaced)
-    (effects (font (size 1.27 1.27)) (justify left bottom))
-  )
   (label "A10" (at 191.135 81.28 0) (fields_autoplaced)
     (effects (font (size 1.27 1.27)) (justify left bottom))
@@
     (effects (font (size 1.27 1.27)) (justify right bottom))
   )
-  (label "P1.4{slash}~{PMGPULSE}" (at 127.635 170.815 0) (fields_autoplaced)
-    (effects (font (size 1.27 1.27)) (justify left bottom))
-  )
   (label "A11" (at 191.135 83.82 0) (fields_autoplaced)
     (effects (font (size 1.27 1.27)) (justify left bottom))
@@
     (effects (font (size 1.27 1.27)) (justify right bottom))
   )
-  (label "P1.5{slash}~{PGMEN}" (at 43.815 81.28 180) (fields_autoplaced)
+  (label "P1.5{slash}~{PGMEN}{slash}MOSI" (at 43.815 81.28 180) (fields_autoplaced)
     (effects (font (size 1.27 1.27)) (justify right bottom))
   )
@@
     (effects (font (size 1.27 1.27)) (justify left bottom))
   )
+  (label "P1.5{slash}~{PGMEN}{slash}MOSI" (at 69.85 78.74 0) (fields_autoplaced)
+    (effects (font (size 1.27 1.27)) (justify left bottom))
+  )
   (label "A14" (at 254 91.44 0) (fields_autoplaced)
     (effects (font (size 1.27 1.27)) (justify left bottom))
@@
     (effects (font (size 1.27 1.27)) (justify left bottom))
   )
+  (label "P1.4{slash}~{PMGPULSE}{slash}~{SS}" (at 69.85 76.2 0) (fields_autoplaced)
+    (effects (font (size 1.27 1.27)) (justify left bottom))
+  )
   (label "D7" (at 375.285 74.93 180) (fields_autoplaced)
     (effects (font (size 1.27 1.27)) (justify right bottom))
@@
     (effects (font (size 1.27 1.27)) (justify right bottom))
   )
+  (label "P1.4{slash}~{PMGPULSE}{slash}~{SS}" (at 124.46 170.815 0) (fields_autoplaced)
+    (effects (font (size 1.27 1.27)) (justify left bottom))
+  )
   (label "ALE" (at 127.635 125.73 0) (fields_autoplaced)
     (effects (font (size 1.27 1.27)) (justify left bottom))
@@
     (effects (font (size 1.27 1.27)) (justify right bottom))
   )
+  (label "P1.6{slash}~{DMA_ACK}{slash}MISO" (at 46.355 210.82 0) (fields_autoplaced)
+    (effects (font (size 1.27 1.27)) (justify left bottom))
+  )
   (label "A10" (at 254 81.28 0) (fields_autoplaced)
     (effects (font (size 1.27 1.27)) (justify left bottom))
@@
     (effects (font (size 1.27 1.27)) (justify left bottom))
   )
-  (label "~{WR}" (at 127.635 165.735 0) (fields_autoplaced)
+  (label "~{WR}" (at 124.46 165.735 0) (fields_autoplaced)
     (effects (font (size 1.27 1.27)) (justify left bottom))
   )
@@
     (effects (font (size 1.27 1.27)) (justify left bottom))
   )
+  (label "P1.6{slash}~{DMA_ACK}{slash}MISO" (at 69.85 81.28 0) (fields_autoplaced)
+    (effects (font (size 1.27 1.27)) (justify left bottom))
+  )
   (label "A4" (at 191.135 66.04 0) (fields_autoplaced)
     (effects (font (size 1.27 1.27)) (justify left bottom))
@@
     (effects (font (size 1.27 1.27)) (justify left bottom))
   )
+  (label "P1.5{slash}~{PGMEN}{slash}MOSI" (at 46.355 208.28 0) (fields_autoplaced)
+    (effects (font (size 1.27 1.27)) (justify left bottom))
+  )
   (label "A6" (at 178.435 88.9 180) (fields_autoplaced)
     (effects (font (size 1.27 1.27)) (justify right bottom))
@@
     (effects (font (size 1.27 1.27)) (justify right bottom))
   )
+  (label "P1.7{slash}~{LTP}{slash}SCK" (at 46.355 205.74 0) (fields_autoplaced)
+    (effects (font (size 1.27 1.27)) (justify left bottom))
+  )
   (label "P1.0" (at 43.815 68.58 180) (fields_autoplaced)
     (effects (font (size 1.27 1.27)) (justify right bottom))
@@
     (effects (font (size 1.27 1.27)) (justify right bottom))
   )
-  (label "P1.6{slash}~{DMA_ACK}" (at 43.815 83.82 180) (fields_autoplaced)
+  (label "P1.6{slash}~{DMA_ACK}{slash}MISO" (at 43.815 83.82 180) (fields_autoplaced)
     (effects (font (size 1.27 1.27)) (justify right bottom))
   )
-  (label "P1.6{slash}~{DMA_ACK}" (at 69.85 81.28 0) (fields_autoplaced)
-    (effects (font (size 1.27 1.27)) (justify left bottom))
-  )
   (label "A2" (at 377.825 82.55 180) (fields_autoplaced)
     (effects (font (size 1.27 1.27)) (justify right bottom))
@@
     (effects (font (size 1.27 1.27)) (justify right bottom))
   )
+  (label "P1.7{slash}~{LTP}{slash}SCK" (at 69.85 83.82 0) (fields_autoplaced)
+    (effects (font (size 1.27 1.27)) (justify left bottom))
+  )
   (label "P3.4{slash}T0" (at 69.85 99.06 0) (fields_autoplaced)
     (effects (font (size 1.27 1.27)) (justify left bottom))
@@
   )
   (symbol (lib_id "Connector:Conn_01x20_Pin") (at 17.78 91.44 0) (unit 1)
-    (in_bom yes) (on_board yes) (dnp no) (fields_autoplaced)
-    (property "Reference" "J2" (at 18.415 68.58 0)
+    (in_bom yes) (on_board yes) (dnp no)
+    (property "Reference" "J2" (at 16.51 67.31 0)
       (effects (font (size 1.27 1.27)))
     )
@@
   )
   (symbol (lib_id "Connector:Conn_01x20_Pin") (at 17.78 143.51 0) (unit 1)
-    (in_bom yes) (on_board yes) (dnp no) (fields_autoplaced)
-    (property "Reference" "J3" (at 18.415 120.65 0)
+    (in_bom yes) (on_board yes) (dnp no)
+    (property "Reference" "J3" (at 15.875 119.38 0)
       (effects (font (size 1.27 1.27)))
     )

Commit message: update
Parts:
- added J4: Conn_02x40_Top_Bottom, Connector_PinHeader_2.54mm:PinHeader_2x40_P2.54mm_Vertical, symbol Connector_Generic:Conn_02x40_Top_Bottom
Connections:
- net A12: now also J4.4 (Pin_4)
- net A13: now also J4.3 (Pin_3)
- net A14: now also J4.2 (Pin_2)
- net A15: now also J4.1 (Pin_1)
Changed lines of the file:
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@@
+    (stroke (width 0) (type default))
+  )
+  (wire (pts (xy 235.585 133.985) (xy 247.015 133.985))
     (stroke (width 0) (type default))
   )
@@
     (stroke (width 0) (type default))
   )
+  (wire (pts (xy 235.585 131.445) (xy 247.015 131.445))
+    (stroke (width 0) (type default))
+  )
   (wire (pts (xy 187.325 71.12) (xy 195.58 71.12))
     (stroke (width 0) (type default))
@@
     (stroke (width 0) (type default))
   )
+  (wire (pts (xy 235.585 139.065) (xy 247.015 139.065))
+    (stroke (width 0) (type default))
+  )
   (wire (pts (xy 334.645 178.435) (xy 344.17 178.435))
     (stroke (width 0) (type default))
@@
     (stroke (width 0) (type default))
   )
+  (wire (pts (xy 235.585 136.525) (xy 247.015 136.525))
+    (stroke (width 0) (type default))
+  )
   (bus (pts (xy 132.08 50.8) (xy 132.08 53.34))
     (stroke (width 0) (type default))
@@
     (effects (font (size 1.27 1.27)) (justify left bottom))
   )
+  (label "A13" (at 235.585 136.525 0) (fields_autoplaced)
+    (effects (font (size 1.27 1.27)) (justify left bottom))
+  )
   (label "D3" (at 287.655 63.5 0) (fields_autoplaced)
     (effects (font (size 1.27 1.27)) (justify left bottom))
@@
     (effects (font (size 1.27 1.27)) (justify right bottom))
   )
+  (label "A12" (at 235.585 139.065 0) (fields_autoplaced)
+    (effects (font (size 1.27 1.27)) (justify left bottom))
+  )
   (label "~{EA}" (at 307.975 77.47 0) (fields_autoplaced)
     (effects (font (size 1.27 1.27)) (justify left bottom))
@@
     (effects (font (size 1.27 1.27)) (justify left bottom))
   )
+  (label "A15" (at 235.585 131.445 0) (fields_autoplaced)
+    (effects (font (size 1.27 1.27)) (justify left bottom))
+  )
   (label "D5" (at 144.145 86.36 180) (fields_autoplaced)
     (effects (font (size 1.27 1.27)) (justify right bottom))
@@
   (label "~{PSEN}" (at 135.255 104.14 180) (fields_autoplaced)
     (effects (font (size 1.27 1.27)) (justify right bottom))
+  )
+  (label "A14" (at 235.585 133.985 0) (fields_autoplaced)
+    (effects (font (size 1.27 1.27)) (justify left bottom))
   )
   (label "A5" (at 191.135 68.58 0) (fields_autoplaced)
@@
         )
       )
+    )
+  )
+  (symbol (lib_id "Connector_Generic:Conn_02x40_Top_Bottom") (at 252.095 179.705 0) (unit 1)
+    (in_bom yes) (on_board yes) (dnp no)
+    (property "Reference" "J4" (at 253.365 150.495 0)
+      (effects (font (size 1.27 1.27)))
+    )
+    (property "Value" "Conn_02x40_Top_Bottom" (at 253.365 233.045 0)
+      (effects (font (size 1.27 1.27)))
+    )
+    (property "Footprint" "Connector_PinHeader_2.54mm:PinHeader_2x40_P2.54mm_Vertical" (at 252.095 179.705 0)
+      (effects (font (size 1.27 1.27)) hide)
+    )
+    (property "Datasheet" "~" (at 252.095 179.705 0)
+      (effects (font (size 1.27 1.27)) hide)
+    )
+    (pin "1")
+    (pin "10")
+    (pin "11")
+    (pin "12")
+    (pin "13")
+    (pin "14")
+    (pin "15")
+    (pin "16")
+    (pin "17")
+    (pin "18")
+    (pin "19")
+    (pin "2")
+    (pin "20")
+    (pin "21")
+    (pin "22")
+    (pin "23")
+    (pin "24")
+    (pin "25")
+    (pin "26")
+    (pin "27")
+    (pin "28")
+    (pin "29")
+    (pin "3")
+    (pin "30")
+    (pin "31")
+    (pin "32")
+    (pin "33")
+    (pin "34")
+    (pin "35")
+    (pin "36")
+    (pin "37")
+    (pin "38")
+    (pin "39")
+    (pin "4")
+    (pin "40")
+    (pin "41")
+    (pin "42")
+    (pin "43")
+    (pin "44")
+    (pin "45")
+    (pin "46")
+    (pin "47")
+    (pin "48")
+    (pin "49")
+    (pin "5")
+    (pin "50")
+    (pin "51")
+    (pin "52")
+    (pin "53")
+    (pin "54")
+    (pin "55")
+    (pin "56")
+    (pin "57")
+    (pin "58")
+    (pin "59")
+    (pin "6")
+    (pin "60")
+    (pin "61")
+    (pin "62")
+    (pin "63")
+    (pin "64")
+    (pin "65")
+    (pin "66")
+    (pin "67")
+    (pin "68")
+    (pin "69")
+    (pin "7")
+    (pin "70")
+    (pin "71")
+    (pin "72")
+    (pin "73")
+    (pin "74")
+    (pin "75")
+    (pin "76")
+    (pin "77")
+    (pin "78")
+    (pin "79")
+    (pin "8")
+    (pin "80")
+    (pin "9")
+    (instances
+      (project "8052-MCU"
+        (path "/e63e39d7-6ac0-4ffd-8aa3-1841a4541b55"
+          (reference "J4") (unit 1)
+        )
+      )
